File: thingamaPRO_abxy/procon_gcc_button_board.kicad_pcb (KiCad board)
At the start: 2 copper layers, 110 x 54.3 mm, 31 parts, among them J1 Button Board, J2 bumpers, SW1 procon_abxy, SW2 procon_dpad, SW3 TL3315NF100Q, SW4 TL3315NF100Q, SW5 TL3315NF100Q, SW6 TL3315NF100Q

Commit message: front board changes
Connections:
- D1 pad 1: BB_BTN_ZR -> BB_BTN_RT
- D1 pad 2: BB_BTN_ZL -> BB_BTN_LT
- SW3 pad 1: (no net) -> BB_BTN_ST
- SW3 pad 4: BB_BTN_ST -> (no net)
- SW5 pad 1: (no net) -> BB_BTN_ST
- SW5 pad 4: BB_BTN_ST -> (no net)
- SW6 pad 1: (no net) -> BB_BTN_ST
- SW6 pad 4: BB_BTN_ST -> (no net)
Routing:
- net BB_BTN_RT: track 68.2 -> 80.6 mm, vias 1 -> 2
- net BB_BTN_ZR: track 79.2 -> 70.1 mm, vias 3 -> 2
- net BB_BTN_ZL: track 71.2 -> 66.0 mm, vias 3 -> 2
- net BB_BTN_LT: track 60.9 -> 63.9 mm
