File: thingamaPRO_abxy/procon_gcc_button_board.kicad_sch (KiCad schematic)
At the start: 24 parts, among them SW5 TL3315NF100Q, SW6 TL3315NF100Q

Commit message: front board changes
Parts:
- D1, D2: value (none) -> BAV70; footprint (none) -> Package_TO_SOT_SMD:SOT-23
- J1: value (none) -> Button Board; footprint (none) -> procon_gcc:molex_5051101492_14P
- J2: value (none) -> bumpers; footprint (none) -> procon_gcc:molex_5051100592_5P
- SW1: value (none) -> procon_abxy; footprint (none) -> procon_gcc:procon_abxy
- SW2: value (none) -> procon_dpad; footprint (none) -> procon_gcc:procon_dpad
- SW3, SW4: value (none) -> TL3315NF100Q; footprint (none) -> procon_gcc:TL3315NFxxxQ
- TP1, TP10, TP11, TP12, TP13, TP14, TP2, TP3, TP4, TP5, TP6, TP7, TP8, TP9: value (none) -> TestPoint; footprint (none) -> TestPoint:TestPoint_Pad_D1.5mm
Connections:
- net BB_BTN_LT: now also D1.2 (A)
- net BB_BTN_RT: now also D1.1 (A)
- net BB_BTN_ZL: no longer D1.2 (A)
- net BB_BTN_ZR: no longer D1.1 (A)
